File: Voltage-display.kicad_sch (KiCad schematic)
At the start: 20 parts, among them J1 Conn_01x02, J2 Conn_01x02, Q1 DMP2035UQ-7, SW1 BD01, U5 PAMC3311QDWERQ1

Commit message: Silenced the erc
Parts:
- removed U5: PAMC3311QDWERQ1, ul_PAMC3311QDWERQ1_footprints:DWE0016A-IPC_A, symbol AMC3311-Q1:PAMC3311QDWERQ1
- added U2: PAMC3311QDWERQ1, ul_PAMC3311QDWERQ1_footprints:DWE0016A-IPC_A, symbol AMC3311-Q1:PAMC3311QDWERQ1
Connections:
- net +5V: now also U2.12 (VDD)
- net DCDC_HV: now also U2.1 (DCDC_OUT), U2.3 (HLDO_IN)
- net DCDC_LV: now also U2.13 (LDO_OUT), U2.16 (DCDC_IN)
- net GND: now also U2.15 (DCDC_GND), U2.9 (GND)
- net HLDO_OUT: now also U2.5 (HLDO_OUT)
- net HV-: now also U2.2 (DCDC_HGND), U2.7 (HGND), U2.8 (HGND)
- net HV_SENSE: now also U2.6 (IN)
- net TC7107_Display/AMC_OUTN: now also U2.10 (OUTN)
- net TC7107_Display/AMC_OUTP: now also U2.11 (OUTP)
Other:
- moved on the sheet: J1

Commit message: Update schematic
Other:
- sheet TC7107_Display ports: added +5V; removed none
Changed lines of the file:
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@@
 	(wire
 		(pts
+			(xy 157.48 127) (xy 190.5 127)
+		)
+		(stroke
+			(width 0)
+			(type default)
+		)
+	)
+	(wire
+		(pts
 			(xy 151.13 55.88) (xy 158.75 55.88)
 		)
@@
 		)
 	)
-	(label "+5V"
-		(at 97.79 34.29 0)
-		(effects
-			(font
-				(size 1.27 1.27)
-			)
-			(justify left bottom)
-		)
-	)
 	(label "HV-"
 		(at 106.68 137.16 180)
@@
 		)
 	)
-	(label "+5V"
-		(at 63.5 127 0)
-		(effects
-			(font
-				(size 1.27 1.27)
-			)
-			(justify left bottom)
-		)
-	)
 	(label "HV_SENSE"
 		(at 106.68 132.08 180)
@@
 	)
 	(symbol
+		(lib_id "power:+5V")
+		(at 63.5 127 270)
+		(unit 1)
+		(body_style 1)
+		(exclude_from_sim no)
+		(in_bom yes)
+		(on_board yes)
+		(in_pos_files yes)
+		(dnp no)
+		(fields_autoplaced yes)
+		(property "Reference" "#PWR01"
+			(at 59.69 127 0)
+			(hide yes)
+			(show_name no)
+			(do_not_autoplace no)
+			(effects
+				(font
+					(size 1.27 1.27)
+				)
+			)
+		)
+		(property "Value" "+5V"
+			(at 67.31 126.9999 90)
+			(show_name no)
+			(do_not_autoplace no)
+			(effects
+				(font
+					(size 1.27 1.27)
+				)
+				(justify left)
+			)
+		)
+		(property "Footprint" ""
+			(at 63.5 127 0)
+			(hide yes)
+			(show_name no)
+			(do_not_autoplace no)
+			(effects
+				(font
+					(size 1.27 1.27)
+				)
+			)
+		)
+		(property "Datasheet" ""
+			(at 63.5 127 0)
+			(hide yes)
+			(show_name no)
+			(do_not_autoplace no)
+			(effects
+				(font
+					(size 1.27 1.27)
+				)
+			)
+		)
+		(property "Description" "Power symbol creates a global label with name \"+5V\""
+			(at 63.5 127 0)
+			(hide yes)
+			(show_name no)
+			(do_not_autoplace no)
+			(effects
+				(font
+					(size 1.27 1.27)
+				)
+			)
+		)
+		(pin "1"
+		)
+		(instances
+			(project "Voltage-display"
+				(path "/aef1bf95-17d0-423a-9dc9-789356babb58"
+					(reference "#PWR01")
+					(unit 1)
+				)
+			)
+		)
+	)
+	(symbol
 		(lib_id "Device:C")
 		(at 88.9 44.45 0)
@@
 	)
 	(symbol
+		(lib_id "power:+5V")
+		(at 97.79 34.29 0)
+		(unit 1)
+		(body_style 1)
+		(exclude_from_sim no)
+		(in_bom yes)
+		(on_board yes)
+		(in_pos_files yes)
+		(dnp no)
+		(fields_autoplaced yes)
+		(property "Reference" "#PWR06"
+			(at 97.79 38.1 0)
+			(hide yes)
+			(show_name no)
+			(do_not_autoplace no)
+			(effects
+				(font
+					(size 1.27 1.27)
+				)
+			)
+		)
+		(property "Value" "+5V"
+			(at 97.79 29.21 0)
+			(show_name no)
+			(do_not_autoplace no)
+			(effects
+				(font
+					(size 1.27 1.27)
+				)
+			)
+		)
+		(property "Footprint" ""
+			(at 97.79 34.29 0)
+			(hide yes)
+			(show_name no)
+			(do_not_autoplace no)
+			(effects
+				(font
+					(size 1.27 1.27)
+				)
+			)
+		)
+		(property "Datasheet" ""
+			(at 97.79 34.29 0)
+			(hide yes)
+			(show_name no)
+			(do_not_autoplace no)
+			(effects
+				(font
+					(size 1.27 1.27)
+				)
+			)
+		)
+		(property "Description" "Power symbol creates a global label with name \"+5V\""
+			(at 97.79 34.29 0)
+			(hide yes)
+			(show_name no)
+			(do_not_autoplace no)
+			(effects
+				(font
+					(size 1.27 1.27)
+				)
+			)
+		)
+		(pin "1"
+		)
+		(instances
+			(project "Voltage-display"
+				(path "/aef1bf95-17d0-423a-9dc9-789356babb58"
+					(reference "#PWR06")
+					(unit 1)
+				)
+			)
+		)
+	)
+	(symbol
 		(lib_id "ul_BD01:BD01")
 		(at 36.83 127 0)
@@
 			(effects
 				(font
+					(size 1.27 1.27)
+				)
+				(justify left)
+			)
+		)
+		(pin "+5V" input
+			(at 190.5 127 180)
+			(effects
+				(font
