File: Voltage-display.kicad_pcb (KiCad board)
At the start: 2 copper layers, 43 parts, among them IC1 TC7107ACPL, J1 HV+ SOLDER, J2 HV- SOLDER, J3 Conn_01x02, Q1 DMP2035UQ-7, U1 AMC1311BQDWVQ1, U2 R05CT05S-R, U3 TC7660SEPA, U4 ADR510ARTZ-REEL7

Commit message: Update files
Parts:
- removed J1: HV+ SOLDER, Connector_Wire:SolderWire-0.5sqmm_1x01_D0.9mm_OD2.1mm_Relief
- removed J2: HV- SOLDER, Connector_Wire:SolderWire-0.5sqmm_1x01_D0.9mm_OD2.1mm_Relief
- added J1 (HV_IN): Conn_01x02, Connector_PinHeader_2.54mm:PinHeader_1x02_P2.54mm_Vertical, F.Cu at (130.5, 102.5)
- added R11: 300, Resistor_SMD:R_1206_3216Metric_Pad1.30x1.75mm_HandSolder, F.Cu at (124.5, 95.5)
- D1: value BZX38450-B2V2-Q -> BZX38450-C2V2-QX
- J2 (5V_IN): renamed from J3
- R4: value 2.8k -> 3k
- moved C10 56.9 mm to (146.1, 106.5), turned to 180 degrees
- moved U3 53.1 mm to (142.2, 102.8), turned to 90 degrees
- moved R10 42.5 mm to (151.4, 65.0)
- moved C11 41.8 mm to (154.0, 95.6), turned to -90 degrees
- moved R9 39.0 mm to (127.5, 86.5)
- moved D1 37.8 mm to (123.5, 87.8), turned to -90 degrees
- moved D2 37.5 mm to (155.1, 69.5)
- moved C12 29.0 mm to (145.0, 92.5), turned to 180 degrees
- moved C13 25.8 mm to (181.0, 114.0), turned to 0 degrees
- moved Q1 25.6 mm to (156.5, 65.9), turned to -90 degrees
- moved AFF3 24.4 mm to (200.2, 82.7), turned to 180 degrees
- moved AFF1 18.0 mm to (200.4, 109.7), turned to 180 degrees
- moved R1 17.5 mm to (130.6, 98.5), turned to 180 degrees
- moved R2 13.1 mm to (130.5, 95.5), turned to 0 degrees
- moved J2 (5V_IN) 10.7 mm to (158.5, 60.5), turned to 90 degrees
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Connections:
- net /+5V_PROTECTED renamed Net-(D2-A2)
- R4 pad 2: Net-(R4-Pad2) -> Net-(R11-Pad1)
Routing:
- net /TC7107_Display/A2: track 75.0 -> 15.3 mm, vias 0 -> 1
- net /TC7107_Display/B2: track 74.5 -> 19.4 mm
- net +5V: track 282.7 -> 234.0 mm
- net /TC7107_Display/G2: track 73.2 -> 29.9 mm, vias 0 -> 2
- net /TC7107_Display/F2: track 41.3 -> 10.1 mm, vias 3 -> 1
- net /TC7107_Display/C2: track 59.1 -> 35.9 mm, vias 1 -> 3
- net /TC7107_Display/E2: track 50.0 -> 33.2 mm, vias 1 -> 3
- net /TC7107_Display/D2: track 47.3 -> 33.2 mm
- net /TC7107_Display/C3: track 58.7 -> 46.6 mm
- net /TC7107_Display/AB4: track 47.0 -> 58.9 mm, vias 2 -> 0
- net /TC7107_Display/A3: track 51.0 -> 40.6 mm, vias 0 -> 4
- net /TC7107_Display/B3: track 37.7 -> 27.7 mm, vias 0 -> 3
- net /TC7107_Display/-5V: track 34.2 -> 24.9 mm, vias 3 -> 1
- net /HV+: track 13.3 -> 4.62 mm
- net /TC7107_Display/D3: track 41.4 -> 33.9 mm, vias 2 -> 3
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
Commit message: changed the footprint for C16 for the BOM
Parts:
- C16: footprint Capacitor_THT:C_Rect_L7.2mm_W7.2mm_P5.00mm_FKS2_FKP2_MKS2_MKP2 -> Capacitor_THT:C_Rect_L7.2mm_W3.0mm_P5.00mm_FKS2_FKP2_MKS2_MKP2
- J1: renamed from J1 (HV_IN)
- J2: renamed from J2 (5V_IN)
Changed lines of the file:
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@@
 		)
 	)
-	(footprint "Capacitor_THT:C_Rect_L7.2mm_W7.2mm_P5.00mm_FKS2_FKP2_MKS2_MKP2"
+	(footprint "Capacitor_THT:C_Rect_L7.2mm_W3.0mm_P5.00mm_FKS2_FKP2_MKS2_MKP2"
 		(layer "F.Cu")
 		(at 151.5 73.5 -90)
-		(descr "C, Rect series, Radial, pin pitch=5.00mm, length*width=7.2*7.2mm^2, Capacitor, http://www.wima.com/EN/WIMA_FKS_2.pdf")
-		(tags "C Rect series Radial pin pitch 5.00mm length 7.2mm width 7.2mm Capacitor")
+		(descr "C, Rect series, Radial, pin pitch=5.00mm, length*width=7.2*3.0mm^2, Capacitor, http://www.wima.com/EN/WIMA_FKS_2.pdf")
+		(tags "C Rect series Radial pin pitch 5.00mm length 7.2mm width 3.0mm Capacitor")
 		(property "Reference" "C16"
-			(at -2.5 -1 180)
+			(at 2.5 -2.75 270)
 			(layer "F.SilkS")
 			(effects
@@
 		)
 		(property "Value" "220nF"
-			(at 2.5 4.85 90)
+			(at 2.5 2.75 270)
 			(layer "F.Fab")
 			(effects
@@
 		)
 		(property "Datasheet" ""
-			(at 0 0 90)
+			(at 0 0 270)
 			(layer "F.Fab")
 			(hide yes)
@@
 		)
 		(property "Description" "Unpolarized capacitor"
-			(at 0 0 90)
+			(at 0 0 270)
 			(layer "F.Fab")
 			(hide yes)
@@
 		)
 		(property "KiLib_Generator" "capacitor/THT/other"
-			(at 0 0 90)
+			(at 0 0 270)
 			(layer "F.SilkS")
 			(hide yes)
@@
 		(duplicate_pad_numbers_are_jumpers no)
 		(fp_line
-			(start -1.22 3.72)
-			(end -1.22 -3.72)
+			(start -1.22 1.62)
+			(end -1.22 -1.62)
 			(stroke
 				(width 0.12)
@@
 		)
 		(fp_line
-			(start 6.22 3.72)
-			(end -1.22 3.72)
+			(start 6.22 1.62)
+			(end -1.22 1.62)
 			(stroke
 				(width 0.12)
@@
 		)
 		(fp_line
-			(start -1.22 -3.72)
-			(end 6.22 -3.72)
+			(start -1.22 -1.62)
+			(end 6.22 -1.62)
 			(stroke
 				(width 0.12)
@@
 		)
 		(fp_line
-			(start 6.22 -3.72)
-			(end 6.22 3.72)
+			(start 6.22 -1.62)
+			(end 6.22 1.62)
 			(stroke
 				(width 0.12)
@@
 		)
 		(fp_rect
-			(start -1.35 -3.85)
-			(end 6.35 3.85)
+			(start -1.35 -1.75)
+			(end 6.35 1.75)
 			(stroke
 				(width 0.05)
@@
 		)
 		(fp_rect
-			(start -1.1 -3.6)
-			(end 6.1 3.6)
+			(start -1.1 -1.5)
+			(end 6.1 1.5)
 			(stroke
 				(width 0.1)
@@
 		)
 		(fp_text user "${REFERENCE}"
-			(at 2.5 0 90)
+			(at 2.5 0 270)
 			(layer "F.Fab")
 			(effects
@@
 		)
 		(embedded_fonts no)
-		(model "${KICAD10_3DMODEL_DIR}/Capacitor_THT.3dshapes/C_Rect_L7.2mm_W7.2mm_P5.00mm_FKS2_FKP2_MKS2_MKP2.step"
+		(model "${KICAD10_3DMODEL_DIR}/Capacitor_THT.3dshapes/C_Rect_L7.2mm_W3.0mm_P5.00mm_FKS2_FKP2_MKS2_MKP2.step"
 			(offset
 				(xyz 0 0 0)
@@
 		(descr "Through hole straight pin header, 1x02, 2.54mm pitch, single row")
 		(tags "Through hole pin header THT 1x02 2.54mm single row")
-		(property "Reference" "J2 (5V_IN)"
+		(property "Reference" "J2"
 			(at 2.5 1.54 180)
 			(layer "F.SilkS")
@@
 		)
 		(property "Value" "100n"
-			(at 0 1.68 90)
+			(at 0.0375 1.68 90)
 			(layer "F.Fab")
 			(effects
@@
 		(descr "Through hole straight pin header, 1x02, 2.54mm pitch, single row")
 		(tags "Through hole pin header THT 1x02 2.54mm single row")
-		(property "Reference" "J1 (HV_IN)"
+		(property "Reference" "J1"
 			(at -6 1.5 0)
 			(layer "F.SilkS")
@@
 	)
 	(segment
+		(start 123 93)
+		(end 123 95.5)
+		(width 0.6)
+		(layer "F.Cu")
+		(net "Net-(R11-Pad1)")
+	)
+	(segment
 		(start 150.5 108)
 		(end 152.46 108)
@@
 	)
 	(segment
+		(start 156.5 69.5)
+		(end 156.5 67.04)
+		(width 0.6)
+		(layer "F.Cu")
+		(net "Net-(D2-A2)")
+	)
+	(segment
+		(start 156.5 67.04)
+		(end 156.46 67)
+		(width 0.6)
+		(layer "F.Cu")
+		(net "Net-(D2-A2)")
+	)
+	(segment
 		(start 154.450002 115.049998)
 		(end 155 114.5)
@@
 		(net "Net-(U3-CAP-)")
 	)
-	(segment
-		(start 156.5 69.5)
-		(end 156.5 67.04)
-		(width 0.6)
-		(layer "F.Cu")
-		(net "Net-(D2-A2)")
-	)
-	(segment
-		(start 156.5 67.04)
-		(end 156.46 67)
-		(width 0.6)
-		(layer "F.Cu")
-		(net "Net-(D2-A2)")
-	)
-	(segment
-		(start 123 93)
-		(end 123 95.5)
-		(width 0.6)
-		(layer "F.Cu")
-		(net "Net-(R11-Pad1)")
-	)
 	(zone

Commit message: Replaced the AMC1311 and RECOME with AMC3311
Parts:
- removed RV2: 500, Potentiometer_THT:Potentiometer_Bourns_3296W_Vertical
- added C2: 1n, Capacitor_SMD:C_0805_2012Metric_Pad1.18x1.45mm_HandSolder, F.Cu at (128.9, 56.0)
- added C3: 1u, Capacitor_SMD:C_1206_3216Metric_Pad1.33x1.80mm_HandSolder, F.Cu at (123.5, 44.7)
- added C4: 1n, Capacitor_SMD:C_0805_2012Metric_Pad1.18x1.45mm_HandSolder, F.Cu at (128.9, 59.0)
- added C5: 1u, Capacitor_SMD:C_1206_3216Metric_Pad1.33x1.80mm_HandSolder, F.Cu at (123.5, 48.0)
- added C6: 1n, Capacitor_SMD:C_0805_2012Metric_Pad1.18x1.45mm_HandSolder, F.Cu at (128.9, 62.0)
- added C7: 100n, Capacitor_SMD:C_1206_3216Metric_Pad1.33x1.80mm_HandSolder, F.Cu at (123.5, 51.4)
- added C8: 100n, Capacitor_SMD:C_1206_3216Metric_Pad1.33x1.80mm_HandSolder, F.Cu at (123.5, 54.7)
- added SW1: BD01, ul_BD01_footprints:SW_BD01_CNK, F.Cu at (133.2, 57.6)
- added U5: PAMC3311QDWERQ1, ul_PAMC3311QDWERQ1_footprints:DWE0016A-IPC_A, F.Cu at (133.6, 48.7)
- R11: value 300 -> 130
- R4: value 3k -> 3.3k
- renumbered C11 to C10, C12 to C11, C13 to C12, C14 to C13, C15 to C14, C16 to C15, C17 to C16, C10 to C9
Connections:
- C1 pad 2: /HV- -> HV-
- IC1 pad 30: /AMC_OUTN -> /TC7107_Display/AMC_OUTN
- IC1 pad 31: /AMCOUTP -> /TC7107_Display/AMC_OUTP
- IC1 pad 32: /AMC_OUTN -> /TC7107_Display/AMC_OUTN
- J1 pad 2: /HV- -> HV-
- R11 pad 2: /HV- -> HV-
Routing:
- added copper zone on F.Cu, net HV-
- removed copper zone on F.Cu, net /HV-

Commit message: Update schematic
Parts:
- removed the C2 at (128.9, 56.0)
- removed the C2 at (128.0, 81.0)
- removed the C3 at (123.5, 44.7)
- removed the C3 at (128.0, 83.5)
- removed the C4 at (146.5, 86.0)
- removed the C4 at (128.9, 59.0)
- removed the C5 at (123.5, 48.0)
- removed the C5 at (146.5, 84.0)
- removed the C6 at (128.9, 62.0)
- removed the C6 at (128.5, 76.0)
- removed the C7 at (127.9, 78.5)
- removed the C7 at (123.5, 51.4)
- removed the C8 at (146.5, 78.0)
- removed the C8 at (123.5, 54.7)
- removed the C9 at (146.5, 81.5)
- removed D1: BZX38450-C2V2-QX, Diode_SMD:D_SOD-323_HandSoldering
- removed R9: 10k, Resistor_SMD:R_1206_3216Metric_Pad1.30x1.75mm_HandSolder
- removed U1: AMC1311BQDWVQ1, ul_AMC1311BQDWVQ1_footprints:DWV8_TEX
- removed U5: PAMC3311QDWERQ1, ul_PAMC3311QDWERQ1_footprints:DWE0016A-IPC_A
- added C2: 1n, Capacitor_SMD:C_0805_2012Metric_Pad1.18x1.45mm_HandSolder, F.Cu at (148.8, 83.4)
- added C3: 1u, Capacitor_SMD:C_1206_3216Metric_Pad1.33x1.80mm_HandSolder, F.Cu at (146.4, 83.2)
- added C4: 1n, Capacitor_SMD:C_0805_2012Metric_Pad1.18x1.45mm_HandSolder, F.Cu at (128.5, 81.0)
- added C5: 1u, Capacitor_SMD:C_1206_3216Metric_Pad1.33x1.80mm_HandSolder, F.Cu at (128.4, 78.0)
- added C6: 1n, Capacitor_SMD:C_0805_2012Metric_Pad1.18x1.45mm_HandSolder, F.Cu at (128.5, 84.0)
- added C7: 100n, Capacitor_SMD:C_1206_3216Metric_Pad1.33x1.80mm_HandSolder, F.Cu at (128.4, 87.0)
- added C8: 100n, Capacitor_SMD:C_1206_3216Metric_Pad1.33x1.80mm_HandSolder, F.Cu at (145.8, 79.2)
- U2: value R05CT05S-R -> PAMC3311QDWERQ1; footprint R05CT055_R_footprints:SMD_16_10.3X7.5X2.6_RCP -> ul_PAMC3311QDWERQ1_footprints:DWE0016A-IPC_A
- moved SW1 28.6 mm to (161.8, 59.5), turned to 180 degrees
- moved R10 16.8 mm to (165.9, 56.5)
- moved D2 15.0 mm to (160.8, 55.6), turned to 180 degrees
- moved J2 14.2 mm to (172.5, 58.0)
- moved Q1 11.3 mm to (166.4, 60.5), turned to 180 degrees
- moved U2 8.52 mm to (138.1, 85.7), turned to 0 degrees
- moved C1 6.79 mm to (133.0, 93.0), turned to -90 degrees
- moved J1 4.98 mm to (127.0, 106.0), turned to 90 degrees
- moved R4 4.92 mm to (128.4, 90.0)
- moved R11 4.09 mm to (123.5, 91.5), turned to -90 degrees
- moved R1 4.08 mm to (128.4, 102.0), turned to 0 degrees
- moved R2 3.23 mm to (128.4, 98.0), turned to 180 degrees
- moved R3 2.50 mm to (128.4, 94.0), turned to 0 degrees
- moved C12 2.22 mm to (179.2, 112.8), turned to 90 degrees
- moved C10 2.06 mm to (153.0, 93.8)
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Connections:
- SW1 pad 2: /+5V -> +5V
- U2 pad 1: +5V -> DCDC_HV
- U2 pad 10: unconnected-(U2-NC-Pad10) -> /TC7107_Display/AMC_OUTN
- U2 pad 11: unconnected-(U2-NC-Pad11) -> /TC7107_Display/AMC_OUTP
- U2 pad 12: unconnected-(U2-NC-Pad12) -> +5V
- U2 pad 13: /ISO_5V -> /DCDC_LV
- U2 pad 14: /ISO_5V -> unconnected-(U2-DIAG-Pad14)
- U2 pad 15: /HV- -> GND
- U2 pad 16: /HV- -> /DCDC_LV
- U2 pad 2: GND -> HV-
- U2 pad 3: +5V -> DCDC_HV
- U2 pad 4: GND -> unconnected-(U2-NC-Pad4)
- U2 pad 5: unconnected-(U2-SYNC_OK-Pad5) -> HLDO_OUT
- U2 pad 6: unconnected-(U2-NC-Pad6) -> /HV_SENSE
- U2 pad 7: unconnected-(U2-NC-Pad7) -> HV-
- U2 pad 8: unconnected-(U2-NC-Pad8) -> HV-
- U2 pad 9: /HV- -> GND
Routing:
- net /AMC_OUTN: track 24.6 -> 0.00 mm, vias 1 -> 0
- net /AMCOUTP: track 19.8 -> 0.00 mm
- net +5V: track 234.0 -> 251.5 mm
- net /ISO_5V: track 16.7 -> 0.00 mm
- net /TC7107_Display/AMC_OUTN: track 0.00 -> 12.6 mm, vias 0 -> 1
- net DCDC_HV: track 0.00 -> 11.5 mm
- net /DCDC_LV: track 0.00 -> 9.16 mm
- net /TC7107_Display/AMC_OUTP: track 0.00 -> 7.26 mm
- net HLDO_OUT: track 0.00 -> 7.02 mm
- net Net-(U1-VIN): track 3.21 -> 0.00 mm
- net /TC7107_Display/-5V: track 24.9 -> 22.5 mm
- net /+5V_IN: track 4.73 -> 6.38 mm
- net Net-(D2-A2): track 2.52 -> 3.92 mm
- net Net-(R2-Pad2): track 2.95 -> 4.00 mm
- net Net-(R1-Pad2): track 3.02 -> 4.00 mm
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- removed copper zone on F.Cu, net GND

Commit message: Update schematic
Parts:
- moved R10 27.3 mm to (143.5, 72.0), turned to 90 degrees
- moved D2 23.9 mm to (147.6, 75.5), turned to 0 degrees
- moved J2 23.1 mm to (151.9, 68.6), turned to 180 degrees
- moved Q1 21.5 mm to (148.0, 71.6), turned to -90 degrees
- moved SW1 16.0 mm to (157.1, 74.8), turned to 90 degrees
- moved R8 9.18 mm to (156.8, 112.5), turned to -90 degrees
- moved C15 7.09 mm to (153.5, 80.5)
- moved R7 4.56 mm to (155.5, 77.6), turned to 180 degrees
- moved C11 4.20 mm to (147.0, 91.0)
- moved AFF3 3.99 mm to (196.9, 80.4)
- moved AFF1 3.91 mm to (196.9, 107.9)
- moved AFF2 3.87 mm to (196.9, 94.2)
- moved U4 3.64 mm to (151.5, 110.5)
- moved R6 3.61 mm to (152.5, 106.0)
- moved C9 2.58 mm to (148.4, 105.5)
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Routing:
- net +5V: track 251.5 -> 223.9 mm, vias 0 -> 4
- net /TC7107_Display/E3: track 51.4 -> 38.2 mm, vias 3 -> 4
- net /TC7107_Display/AMC_OUTP: track 7.26 -> 19.8 mm
- net /TC7107_Display/AMC_OUTN: track 12.6 -> 24.9 mm
- net /TC7107_Display/E2: track 33.2 -> 21.7 mm, vias 3 -> 2
- net Net-(D2-A2): track 3.92 -> 13.2 mm
- net /TC7107_Display/G2: track 29.9 -> 22.5 mm, vias 2 -> 1
- net /TC7107_Display/F2: track 10.1 -> 17.1 mm, vias 1 -> 2
- net /TC7107_Display/AB4: track 58.9 -> 52.5 mm, vias 0 -> 1
- net GND: track 2.23 -> 7.75 mm, vias 2 -> 7
- net /TC7107_Display/V_BUFF: track 12.1 -> 7.04 mm
- net /TC7107_Display/C3: track 46.6 -> 41.8 mm
- net HV-: track 0.00 -> 4.02 mm, vias 0 -> 2
- net /TC7107_Display/OSC1: track 8.20 -> 4.47 mm
- net /TC7107_Display/-5V: track 22.5 -> 25.5 mm, vias 1 -> 3
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- added copper zone on F.Cu, net GND
Other:
- board outline added: 81.5 x 53.5 mm
